File: pcb/LeftRightMapping.kicad_sch (KiCad schematic)
At the start: 7 parts

Commit message: Placing more components onto the PCB and removing more stale leftovers from the now absent Rotary Encoder.
Parts:
- removed JP7: SolderJumper_2_Open, Jumper:SolderJumper-2_P1.3mm_Open_TrianglePad1.0x1.5mm, symbol Jumper:SolderJumper_2_Open
Changed lines of the file:
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@@
 	(wire
 		(pts
-			(xy 92.71 111.76) (xy 113.03 111.76)
+			(xy 92.71 54.61) (xy 113.03 54.61)
 		)
 		(stroke
@@
 	(wire
 		(pts
-			(xy 120.65 111.76) (xy 137.16 111.76)
+			(xy 92.71 77.47) (xy 113.03 77.47)
 		)
 		(stroke
@@
 		)
 	)
-	(wire
-		(pts
-			(xy 92.71 54.61) (xy 113.03 54.61)
-		)
-		(stroke
-			(width 0)
-			(type default)
-		)
-	)
-	(wire
-		(pts
-			(xy 92.71 77.47) (xy 113.03 77.47)
-		)
-		(stroke
-			(width 0)
-			(type default)
-		)
-	)
 	(hierarchical_label "R_COL_3"
 		(shape input)
@@
 		)
 	)
-	(hierarchical_label "R_ROW_4"
-		(shape input)
-		(at 137.16 111.76 0)
-		(fields_autoplaced yes)
-		(effects
-			(font
-				(size 1.27 1.27)
-			)
-			(justify left)
-		)
-	)
 	(hierarchical_label "R_ROW_2"
 		(shape input)
@@
 		(shape input)
 		(at 92.71 66.04 180)
-		(fields_autoplaced yes)
-		(effects
-			(font
-				(size 1.27 1.27)
-			)
-			(justify right)
-		)
-	)
-	(hierarchical_label "ROW_4"
-		(shape input)
-		(at 92.71 111.76 180)
 		(fields_autoplaced yes)
 		(effects
@@
 					(unit 1)
 				)
-			)
-		)
-	)
-	(symbol
-		(lib_id "Jumper:SolderJumper_2_Open")
-		(at 116.84 111.76 0)
-		(unit 1)
-		(exclude_from_sim no)
-		(in_bom yes)
-		(on_board yes)
-		(dnp no)
-		(fields_autoplaced yes)
-		(property "Reference" "JP7"
-			(at 116.84 105.41 0)
-			(effects
-				(font
-					(size 1.27 1.27)
-				)
-			)
-		)
-		(property "Value" "SolderJumper_2_Open"
-			(at 116.84 107.95 0)
-			(effects
-				(font
-					(size 1.27 1.27)
-				)
-			)
-		)
-		(property "Footprint" "Jumper:SolderJumper-2_P1.3mm_Open_TrianglePad1.0x1.5mm"
-			(at 116.84 111.76 0)
-			(effects
-				(font
-					(size 1.27 1.27)
-				)
-				(hide yes)
-			)
-		)
-		(property "Datasheet" "~"
-			(at 116.84 111.76 0)
-			(effects
-				(font
-					(size 1.27 1.27)
-				)
-				(hide yes)
-			)
-		)
-		(property "Description" ""
-			(at 116.84 111.76 0)
-			(effects
-				(font
-					(size 1.27 1.27)
-				)
-				(hide yes)
-			)
-		)
-		(pin "1"
-		)
-		(pin "2"
-		)
-		(instances
-			(project "cheapino"
-				(path "/9203b006-47ac-4f34-8cc4-2b709e3df56f/7b8b7eaa-434c-41c6-a017-c1171f20f2be"
-					(reference "JP7")
-					(unit 1)
-				)
