File: pcb/ExtConnectors.kicad_sch (KiCad schematic)
At the start: 12 parts, among them J1 USB_C_Receptacle_USB2.0_16P, J2 DBG, J3 AudioJack4, U2 TPD2E2U06, U3 AP2112K-3.3, U6 TVS0500DRV, U9 TPD2E2U06

Commit message: Adding reversible MX Sockets and SK6812MiniE footprints, finishing the replacement of Ethernet with a TRRS connector and selectable 0Ohm resistors to swap Rx/Tx for the interconnect.
Parts:
- removed J3: AudioJack4, symbol Connector_Audio:AudioJack4
- added D43: SK34A-LTP, Diode_SMD:D_SMA_Handsoldering, symbol Device:D_Schottky
- added J3: SJ-43514, Extra:CUI_SJ-43514, symbol Extra:SJ-43514
- added R14: 5k6, Resistor_SMD:R_0805_2012Metric_Pad1.20x1.40mm_HandSolder, symbol Device:R
- added R15: 10k, Resistor_SMD:R_0805_2012Metric_Pad1.20x1.40mm_HandSolder, symbol Device:R
- added R16, R17, R18, R19: 0, Resistor_SMD:R_0805_2012Metric_Pad1.20x1.40mm_HandSolder, symbol Device:R
- renumbered U6 to U4, U2 to U5, U9 to U6
Connections:
- net GND: now also J3.1, R15.2; no longer U5.1 (NC), U5.2 (NC)
- net UART_Rx: now also R16.2, R19.2
- net UART_Tx: now also R17.2, R18.2
- net VBUS: now also D43.2 (A), R14.1; no longer C1.1, R3.2, U3.1 (VIN)
- new net Interconnect_Signal1: J3.3, R16.1, R18.1
- new net Interconnect_Signal2: J3.4, R17.1, R19.1
- new net VBUS_Sense: R14.2, R15.1
- new net VSYS: C1.1, D43.1 (K), J3.2, R3.2, U3.1 (VIN)
Other:
- note added: "ESD protection on non-USB half?"
- note added: "Install one pair of R16/R17 or R18/R19 Alternate between the two halves"
- note added: "Total power draw via USB for LEDs at peak ~45mA per ((18+6)*2) = 2.16A 80% of 3A => 2.4A, 240mA for the rest of the board with 3A/5V input USB supply"
- moved on the sheet: U4

Commit message: Renumbering all reference designations and adding an initial layout for each keyswtich sub-pcb.
Parts:
- renumbered C1 to C15, C2 to C16, D43 to D61, R14 to R10, R15 to R11, R16 to R12, R17 to R13, R18 to R14, R19 to R15, R1 to R7, R2 to R8, R3 to R9
Other:
- note added: "Install one pair of R12/R13 or R14/R15 Alternate between the two halves"
- note removed: "Install one pair of R16/R17 or R18/R19 Alternate between the two halves"
Changed lines of the file:
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@@
 		)
 	)
-	(text "Install one pair of R16/R17 or R18/R19\nAlternate between the two halves"
+	(text "Install one pair of R12/R13 or R14/R15\nAlternate between the two halves"
 		(exclude_from_sim no)
 		(at 86.614 145.796 0)
@@
 		(dnp no)
 		(fields_autoplaced yes)
-		(property "Reference" "R18"
+		(property "Reference" "R14"
 			(at 102.87 153.67 90)
 			(effects
@@
 			(project "cheapino"
 				(path "/9203b006-47ac-4f34-8cc4-2b709e3df56f/e6ab333d-5f1a-4b76-81c6-498aebdc0c3b"
-					(reference "R18")
+					(reference "R14")
 					(unit 1)
 				)
@@
 		(dnp no)
 		(fields_autoplaced yes)
-		(property "Reference" "R14"
+		(property "Reference" "R10"
 			(at 88.9 59.6899 0)
 			(effects
@@
 			(project "cheapino"
 				(path "/9203b006-47ac-4f34-8cc4-2b709e3df56f/e6ab333d-5f1a-4b76-81c6-498aebdc0c3b"
-					(reference "R14")
+					(reference "R10")
 					(unit 1)
 				)
@@
 		(dnp no)
 		(fields_autoplaced yes)
-		(property "Reference" "R1"
+		(property "Reference" "R7"
 			(at 190.5 87.63 90)
 			(effects
@@
 			(project ""
 				(path "/9203b006-47ac-4f34-8cc4-2b709e3df56f/e6ab333d-5f1a-4b76-81c6-498aebdc0c3b"
-					(reference "R1")
+					(reference "R7")
 					(unit 1)
 				)
@@
 		(on_board yes)
 		(dnp no)
-		(property "Reference" "R2"
+		(property "Reference" "R8"
 			(at 190.5 96.52 90)
 			(effects
@@
 			(project "cheapino"
 				(path "/9203b006-47ac-4f34-8cc4-2b709e3df56f/e6ab333d-5f1a-4b76-81c6-498aebdc0c3b"
-					(reference "R2")
+					(reference "R8")
 					(unit 1)
 				)
@@
 		(dnp no)
 		(fields_autoplaced yes)
-		(property "Reference" "R16"
+		(property "Reference" "R12"
 			(at 102.87 119.38 90)
 			(effects
@@
 			(project ""
 				(path "/9203b006-47ac-4f34-8cc4-2b709e3df56f/e6ab333d-5f1a-4b76-81c6-498aebdc0c3b"
-					(reference "R16")
+					(reference "R12")
 					(unit 1)
 				)
@@
 		(dnp no)
 		(fields_autoplaced yes)
-		(property "Reference" "R15"
+		(property "Reference" "R11"
 			(at 88.9 67.3099 0)
 			(effects
@@
 			(project "cheapino"
 				(path "/9203b006-47ac-4f34-8cc4-2b709e3df56f/e6ab333d-5f1a-4b76-81c6-498aebdc0c3b"
-					(reference "R15")
+					(reference "R11")
 					(unit 1)
 				)
@@
 		(on_board yes)
 		(dnp no)
-		(property "Reference" "R3"
+		(property "Reference" "R9"
 			(at 234.95 53.3401 0)
 			(effects
@@
 			(project ""
 				(path "/9203b006-47ac-4f34-8cc4-2b709e3df56f/e6ab333d-5f1a-4b76-81c6-498aebdc0c3b"
-					(reference "R3")
+					(reference "R9")
 					(unit 1)
 				)
@@
 		(dnp no)
 		(fields_autoplaced yes)
-		(property "Reference" "R19"
+		(property "Reference" "R15"
 			(at 102.87 163.83 90)
 			(effects
@@
 			(project "cheapino"
 				(path "/9203b006-47ac-4f34-8cc4-2b709e3df56f/e6ab333d-5f1a-4b76-81c6-498aebdc0c3b"
-					(reference "R19")
+					(reference "R15")
 					(unit 1)
 				)
@@
 		(on_board yes)
 		(dnp no)
-		(property "Reference" "C1"
+		(property "Reference" "C15"
 			(at 222.25 50.7999 0)
 			(effects
@@
 			(project ""
 				(path "/9203b006-47ac-4f34-8cc4-2b709e3df56f/e6ab333d-5f1a-4b76-81c6-498aebdc0c3b"
-					(reference "C1")
+					(reference "C15")
 					(unit 1)
 				)
@@
 		(dnp no)
 		(fields_autoplaced yes)
-		(property "Reference" "C2"
+		(property "Reference" "C16"
 			(at 267.97 50.7999 0)
 			(effects
@@
 			(project "cheapino"
 				(path "/9203b006-47ac-4f34-8cc4-2b709e3df56f/e6ab333d-5f1a-4b76-81c6-498aebdc0c3b"
-					(reference "C2")
+					(reference "C16")
 					(unit 1)
 				)
@@
 		(dnp no)
 		(fields_autoplaced yes)
-		(property "Reference" "R17"
+		(property "Reference" "R13"
 			(at 102.87 129.54 90)
 			(effects
@@
 			(project "cheapino"
 				(path "/9203b006-47ac-4f34-8cc4-2b709e3df56f/e6ab333d-5f1a-4b76-81c6-498aebdc0c3b"
-					(reference "R17")
+					(reference "R13")
 					(unit 1)
 				)
@@
 		(on_board yes)
 		(dnp no)
-		(property "Reference" "D43"
+		(property "Reference" "D61"
 			(at 200.9775 41.91 0)
 			(effects
@@
 			(project ""
 				(path "/9203b006-47ac-4f34-8cc4-2b709e3df56f/e6ab333d-5f1a-4b76-81c6-498aebdc0c3b"
-					(reference "D43")
-					(unit 1)
-				)
+					(reference "D61")
+					(unit 1)
+				)
