File: pcb/micro.kicad_sch (KiCad schematic)
At the start: 25 parts, among them SW1 BOOT, SW2 RST, U1 RP2040, U2 W25Q128JVSIQ, Y1 12MHz

Commit message: Renumbering all reference designations and adding an initial layout for each keyswtich sub-pcb.
Parts:
- renumbered C12 to C1, C8 to C10, C14 to C12, C15 to C13, C16 to C14, C13 to C2, C9 to C3, C10 to C4, C3 to C5, C4 to C6, C5 to C7, C6 to C8, C7 to C9, R9 to R1, R8 to R2, R7 to R3, R6 to R4, R4 to R6
Changed lines of the file:
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@@
 		(dnp no)
 		(fields_autoplaced yes)
-		(property "Reference" "C4"
+		(property "Reference" "C6"
 			(at 195.58 31.7499 0)
 			(effects
@@
 			(project "cheapino"
 				(path "/9203b006-47ac-4f34-8cc4-2b709e3df56f/b2f85b86-5933-4a5f-88c2-315afb4ca3cd"
-					(reference "C4")
+					(reference "C6")
 					(unit 1)
 				)
@@
 		(dnp no)
 		(fields_autoplaced yes)
-		(property "Reference" "C9"
+		(property "Reference" "C3"
 			(at 229.87 57.1499 0)
 			(effects
@@
 			(project "cheapino"
 				(path "/9203b006-47ac-4f34-8cc4-2b709e3df56f/b2f85b86-5933-4a5f-88c2-315afb4ca3cd"
-					(reference "C9")
+					(reference "C3")
 					(unit 1)
 				)
@@
 		(dnp no)
 		(fields_autoplaced yes)
-		(property "Reference" "C10"
+		(property "Reference" "C4"
 			(at 201.93 49.5299 0)
 			(effects
@@
 			(project "cheapino"
 				(path "/9203b006-47ac-4f34-8cc4-2b709e3df56f/b2f85b86-5933-4a5f-88c2-315afb4ca3cd"
-					(reference "C10")
+					(reference "C4")
 					(unit 1)
 				)
@@
 		(dnp no)
 		(fields_autoplaced yes)
-		(property "Reference" "C12"
+		(property "Reference" "C1"
 			(at 214.63 74.9299 0)
 			(effects
@@
 			(project "cheapino"
 				(path "/9203b006-47ac-4f34-8cc4-2b709e3df56f/b2f85b86-5933-4a5f-88c2-315afb4ca3cd"
-					(reference "C12")
+					(reference "C1")
 					(unit 1)
 				)
@@
 		(dnp no)
 		(fields_autoplaced yes)
-		(property "Reference" "R4"
+		(property "Reference" "R6"
 			(at 121.92 49.5299 0)
 			(effects
@@
 			(project ""
 				(path "/9203b006-47ac-4f34-8cc4-2b709e3df56f/b2f85b86-5933-4a5f-88c2-315afb4ca3cd"
-					(reference "R4")
+					(reference "R6")
 					(unit 1)
 				)
@@
 		(dnp no)
 		(fields_autoplaced yes)
-		(property "Reference" "C7"
+		(property "Reference" "C9"
 			(at 233.68 31.7499 0)
 			(effects
@@
 			(project "cheapino"
 				(path "/9203b006-47ac-4f34-8cc4-2b709e3df56f/b2f85b86-5933-4a5f-88c2-315afb4ca3cd"
-					(reference "C7")
+					(reference "C9")
 					(unit 1)
 				)
@@
 		(dnp no)
 		(fields_autoplaced yes)
-		(property "Reference" "R6"
+		(property "Reference" "R4"
 			(at 69.85 58.42 90)
 			(effects
@@
 			(project "cheapino"
 				(path "/9203b006-47ac-4f34-8cc4-2b709e3df56f/b2f85b86-5933-4a5f-88c2-315afb4ca3cd"
-					(reference "R6")
+					(reference "R4")
 					(unit 1)
 				)
@@
 		(dnp no)
 		(fields_autoplaced yes)
-		(property "Reference" "C15"
+		(property "Reference" "C13"
 			(at 68.58 88.9 90)
 			(effects
@@
 			(project "cheapino"
 				(path "/9203b006-47ac-4f34-8cc4-2b709e3df56f/b2f85b86-5933-4a5f-88c2-315afb4ca3cd"
-					(reference "C15")
+					(reference "C13")
 					(unit 1)
 				)
@@
 		(dnp no)
 		(fields_autoplaced yes)
-		(property "Reference" "C16"
+		(property "Reference" "C14"
 			(at 118.11 148.5899 0)
 			(effects
@@
 			(project "cheapino"
 				(path "/9203b006-47ac-4f34-8cc4-2b709e3df56f/b2f85b86-5933-4a5f-88c2-315afb4ca3cd"
-					(reference "C16")
+					(reference "C14")
 					(unit 1)
 				)
@@
 		(dnp no)
 		(fields_autoplaced yes)
-		(property "Reference" "R9"
+		(property "Reference" "R1"
 			(at 73.66 142.24 90)
 			(effects
@@
 			(project ""
 				(path "/9203b006-47ac-4f34-8cc4-2b709e3df56f/b2f85b86-5933-4a5f-88c2-315afb4ca3cd"
-					(reference "R9")
+					(reference "R1")
 					(unit 1)
 				)
@@
 		(dnp no)
 		(fields_autoplaced yes)
-		(property "Reference" "C14"
+		(property "Reference" "C12"
 			(at 68.58 105.41 90)
 			(effects
@@
 			(project ""
 				(path "/9203b006-47ac-4f34-8cc4-2b709e3df56f/b2f85b86-5933-4a5f-88c2-315afb4ca3cd"
-					(reference "C14")
+					(reference "C12")
 					(unit 1)
 				)
@@
 		(dnp no)
 		(fields_autoplaced yes)
-		(property "Reference" "C8"
+		(property "Reference" "C10"
 			(at 246.38 31.7499 0)
 			(effects
@@
 			(project "cheapino"
 				(path "/9203b006-47ac-4f34-8cc4-2b709e3df56f/b2f85b86-5933-4a5f-88c2-315afb4ca3cd"
-					(reference "C8")
+					(reference "C10")
 					(unit 1)
 				)
@@
 		(dnp no)
 		(fields_autoplaced yes)
-		(property "Reference" "R8"
+		(property "Reference" "R2"
 			(at 88.9 148.5899 0)
 			(effects
@@
 			(project ""
 				(path "/9203b006-47ac-4f34-8cc4-2b709e3df56f/b2f85b86-5933-4a5f-88c2-315afb4ca3cd"
-					(reference "R8")
+					(reference "R2")
 					(unit 1)
 				)
@@
 		(dnp no)
 		(fields_autoplaced yes)
-		(property "Reference" "C13"
+		(property "Reference" "C2"
 			(at 227.33 74.9299 0)
 			(effects
@@
 			(project "cheapino"
 				(path "/9203b006-47ac-4f34-8cc4-2b709e3df56f/b2f85b86-5933-4a5f-88c2-315afb4ca3cd"
-					(reference "C13")
+					(reference "C2")
 					(unit 1)
 				)
@@
 		(dnp no)
 		(fields_autoplaced yes)
-		(property "Reference" "C3"
+		(property "Reference" "C5"
 			(at 182.88 31.7499 0)
 			(effects
@@
 			(project ""
 				(path "/9203b006-47ac-4f34-8cc4-2b709e3df56f/b2f85b86-5933-4a5f-88c2-315afb4ca3cd"
-					(reference "C3")
+					(reference "C5")
 					(unit 1)
 				)
@@
 		(dnp no)
 		(fields_autoplaced yes)
-		(property "Reference" "R7"
+		(property "Reference" "R3"
 			(at 115.57 104.14 90)
 			(effects
@@
 			(project ""
 				(path "/9203b006-47ac-4f34-8cc4-2b709e3df56f/b2f85b86-5933-4a5f-88c2-315afb4ca3cd"
-					(reference "R7")
+					(reference "R3")
 					(unit 1)
 				)
@@
 		(dnp no)
 		(fields_autoplaced yes)
-		(property "Reference" "C6"
+		(property "Reference" "C8"
 			(at 220.98 31.7499 0)
 			(effects
@@
 			(project "cheapino"
 				(path "/9203b006-47ac-4f34-8cc4-2b709e3df56f/b2f85b86-5933-4a5f-88c2-315afb4ca3cd"
-					(reference "C6")
+					(reference "C8")
 					(unit 1)
 				)
@@
 		(dnp no)
 		(fields_autoplaced yes)
-		(property "Reference" "C5"
+		(property "Reference" "C7"
 			(at 208.28 31.7499 0)
 			(effects
@@
 			(project "cheapino"
 				(path "/9203b006-47ac-4f34-8cc4-2b709e3df56f/b2f85b86-5933-4a5f-88c2-315afb4ca3cd"
-					(reference "C5")
+					(reference "C7")
 					(unit 1)
 				)
